File: ECAD/antenna.kicad_sch (KiCad schematic)
At the start: 16 parts

Commit message: Updated schmatics
Parts:
- AE1: footprint Connector_JST:JST_XH_B2B-XH-AM_1x02_P2.50mm_Vertical -> Connector_JST:JST_PH_B2B-PH-K_1x02_P2.00mm_Vertical
- C0A1: renamed from C10; footprint Capacitor_SMD:C_01005_0402Metric -> Capacitor_SMD:C_0805_2012Metric
- C0B1: renamed from C11; footprint Capacitor_SMD:C_01005_0402Metric -> Capacitor_SMD:C_0805_2012Metric
- C1A1: renamed from C12; value Matching -> tbd; footprint Capacitor_SMD:C_01005_0402Metric -> Capacitor_SMD:C_0805_2012Metric
- C1D1: renamed from C13; value Matching -> tbd; footprint Capacitor_SMD:C_01005_0402Metric -> Capacitor_SMD:C_0805_2012Metric
- C2B1: renamed from C14; value Matching -> tbd; footprint Capacitor_SMD:C_01005_0402Metric -> Capacitor_SMD:C_0805_2012Metric
- C2D1: renamed from C15; value Matching -> tbd; footprint Capacitor_SMD:C_01005_0402Metric -> Capacitor_SMD:C_0805_2012Metric
- C3A1: renamed from C18; footprint Capacitor_SMD:C_01005_0402Metric -> Capacitor_SMD:C_0805_2012Metric
- C3B1: renamed from C16; footprint Capacitor_SMD:C_01005_0402Metric -> Capacitor_SMD:C_0805_2012Metric
- C8: renamed from C20; footprint Capacitor_SMD:C_01005_0402Metric -> Capacitor_SMD:C_0805_2012Metric
- CANT1: renamed from C19; value Cant -> tbd; footprint Capacitor_SMD:C_01005_0402Metric -> Capacitor_SMD:C_0805_2012Metric
- CANT2: renamed from C17; value Cant -> tbd; footprint Capacitor_SMD:C_01005_0402Metric -> Capacitor_SMD:C_0805_2012Metric
- L0A1: renamed from L1; footprint Inductor_SMD:L_2010_5025Metric -> Inductor_SMD:L_0805_2012Metric
- L0B1: renamed from L2; footprint Inductor_SMD:L_2010_5025Metric -> Inductor_SMD:L_0805_2012Metric
- R1A1: renamed from R7; footprint Resistor_SMD:R_01005_0402Metric -> Resistor_SMD:R_0805_2012Metric
- R1B1: renamed from R9; footprint Resistor_SMD:R_01005_0402Metric -> Resistor_SMD:R_0805_2012Metric
Changed lines of the file:
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@@
 		(on_board yes)
 		(dnp no)
-		(property "Reference" "C19"
+		(property "Reference" "CANT1"
 			(at 122.682 51.308 0)
 			(effects
@@
 			)
 		)
-		(property "Value" "Cant"
+		(property "Value" "tbd"
 			(at 124.714 51.308 0)
 			(effects
@@
 			)
 		)
-		(property "Footprint" "Capacitor_SMD:C_01005_0402Metric"
+		(property "Footprint" "Capacitor_SMD:C_0805_2012Metric"
 			(at 123.19 51.1048 0)
 			(effects
@@
 			(project "RFID_Reader"
 				(path "/4670be35-0898-46f4-be4d-f086d3203cc5/68791068-2e08-46a9-8a2f-80be28f652d5"
-					(reference "C19")
+					(reference "CANT1")
 					(unit 1)
 				)
@@
 		(on_board yes)
 		(dnp no)
-		(property "Reference" "C12"
+		(property "Reference" "C1A1"
 			(at 110.998 62.484 90)
 			(effects
@@
 			)
 		)
-		(property "Value" "Matching"
+		(property "Value" "tbd"
 			(at 110.998 65.024 90)
 			(effects
@@
 			)
 		)
-		(property "Footprint" "Capacitor_SMD:C_01005_0402Metric"
+		(property "Footprint" "Capacitor_SMD:C_0805_2012Metric"
 			(at 113.03 68.8848 0)
 			(effects
@@
 			(project "RFID_Reader"
 				(path "/4670be35-0898-46f4-be4d-f086d3203cc5/68791068-2e08-46a9-8a2f-80be28f652d5"
-					(reference "C12")
+					(reference "C1A1")
 					(unit 1)
 				)
@@
 		(on_board yes)
 		(dnp no)
-		(property "Reference" "R7"
+		(property "Reference" "R1A1"
 			(at 97.536 61.468 90)
 			(effects
@@
 			)
 		)
-		(property "Footprint" "Resistor_SMD:R_01005_0402Metric"
+		(property "Footprint" "Resistor_SMD:R_0805_2012Metric"
 			(at 105.918 62.23 90)
 			(effects
@@
 			(project "RFID_Reader"
 				(path "/4670be35-0898-46f4-be4d-f086d3203cc5/68791068-2e08-46a9-8a2f-80be28f652d5"
-					(reference "R7")
+					(reference "R1A1")
 					(unit 1)
 				)
@@
 		(on_board yes)
 		(dnp no)
-		(property "Reference" "C13"
+		(property "Reference" "C1D1"
 			(at 110.49 100.33 90)
 			(effects
@@
 			)
 		)
-		(property "Value" "Matching"
+		(property "Value" "tbd"
 			(at 110.49 102.362 90)
 			(effects
@@
 			)
 		)
-		(property "Footprint" "Capacitor_SMD:C_01005_0402Metric"
+		(property "Footprint" "Capacitor_SMD:C_0805_2012Metric"
 			(at 114.3 95.5548 0)
 			(effects
@@
 			(project "RFID_Reader"
 				(path "/4670be35-0898-46f4-be4d-f086d3203cc5/68791068-2e08-46a9-8a2f-80be28f652d5"
-					(reference "C13")
+					(reference "C1D1")
 					(unit 1)
 				)
@@
 		(dnp no)
 		(fields_autoplaced yes)
-		(property "Reference" "C14"
+		(property "Reference" "C2B1"
 			(at 120.65 74.9299 0)
 			(effects
@@
 			)
 		)
-		(property "Value" "Matching"
+		(property "Value" "tbd"
 			(at 120.65 77.4699 0)
 			(effects
@@
 			)
 		)
-		(property "Footprint" "Capacitor_SMD:C_01005_0402Metric"
+		(property "Footprint" "Capacitor_SMD:C_0805_2012Metric"
 			(at 115.8748 72.39 0)
 			(effects
@@
 			(project "RFID_Reader"
 				(path "/4670be35-0898-46f4-be4d-f086d3203cc5/68791068-2e08-46a9-8a2f-80be28f652d5"
-					(reference "C14")
+					(reference "C2B1")
 					(unit 1)
 				)
@@
 		(on_board yes)
 		(dnp no)
-		(property "Reference" "C16"
+		(property "Reference" "C3B1"
 			(at 77.978 101.346 90)
 			(effects
@@
 			)
 		)
-		(property "Footprint" "Capacitor_SMD:C_01005_0402Metric"
+		(property "Footprint" "Capacitor_SMD:C_0805_2012Metric"
 			(at 76.2 106.3752 0)
 			(effects
@@
 			(project "RFID_Reader"
 				(path "/4670be35-0898-46f4-be4d-f086d3203cc5/68791068-2e08-46a9-8a2f-80be28f652d5"
-					(reference "C16")
+					(reference "C3B1")
 					(unit 1)
 				)
@@
 		(on_board yes)
 		(dnp no)
-		(property "Reference" "C15"
+		(property "Reference" "C2D1"
 			(at 119.888 87.884 0)
 			(effects
@@
 			)
 		)
-		(property "Value" "Matching"
+		(property "Value" "tbd"
 			(at 119.888 89.916 0)
 			(effects
@@
 			)
 		)
-		(property "Footprint" "Capacitor_SMD:C_01005_0402Metric"
+		(property "Footprint" "Capacitor_SMD:C_0805_2012Metric"
 			(at 115.8748 87.63 0)
 			(effects
@@
 			(project "RFID_Reader"
 				(path "/4670be35-0898-46f4-be4d-f086d3203cc5/68791068-2e08-46a9-8a2f-80be28f652d5"
-					(reference "C15")
+					(reference "C2D1")
 					(unit 1)
 				)
@@
 		(on_board yes)
 		(dnp no)
-		(property "Reference" "C10"
+		(property "Reference" "C0A1"
 			(at 94.488 76.454 0)
 			(effects
@@
 			)
 		)
-		(property "Footprint" "Capacitor_SMD:C_01005_0402Metric"
+		(property "Footprint" "Capacitor_SMD:C_0805_2012Metric"
 			(at 102.5652 81.28 0)
 			(effects
@@
 			(project "RFID_Reader"
 				(path "/4670be35-0898-46f4-be4d-f086d3203cc5/68791068-2e08-46a9-8a2f-80be28f652d5"
-					(reference "C10")
+					(reference "C0A1")
 					(unit 1)
 				)
@@
 			)
 		)
-		(property "Footprint" "Connector_JST:JST_XH_B2B-XH-AM_1x02_P2.50mm_Vertical"
+		(property "Footprint" "Connector_JST:JST_PH_B2B-PH-K_1x02_P2.00mm_Vertical"
 			(at 138.43 82.55 0)
 			(effects
@@
 		(on_board yes)
 		(dnp no)
-		(property "Reference" "C18"
+		(property "Reference" "C3A1"
 			(at 77.978 61.214 90)
 			(effects
@@
 			)
 		)
-		(property "Footprint" "Capacitor_SMD:C_01005_0402Metric"
+		(property "Footprint" "Capacitor_SMD:C_0805_2012Metric"
 			(at 76.2 56.1848 0)
 			(effects
@@
 			(project "RFID_Reader"
 				(path "/4670be35-0898-46f4-be4d-f086d3203cc5/68791068-2e08-46a9-8a2f-80be28f652d5"
-					(reference "C18")
+					(reference "C3A1")
 					(unit 1)
 				)
@@
 		(on_board yes)
 		(dnp no)
-		(property "Reference" "L1"
+		(property "Reference" "L0A1"
 			(at 88.9 67.31 90)
 			(effects
@@
 			)
 		)
-		(property "Footprint" "Inductor_SMD:L_2010_5025Metric"
+		(property "Footprint" "Inductor_SMD:L_0805_2012Metric"
 			(at 90.17 72.39 0)
 			(effects
@@
 			(project "RFID_Reader"
 				(path "/4670be35-0898-46f4-be4d-f086d3203cc5/68791068-2e08-46a9-8a2f-80be28f652d5"
-					(reference "L1")
+					(reference "L0A1")
 					(unit 1)
 				)
@@
 		(on_board yes)
 		(dnp no)
-		(property "Reference" "C20"
-			(at 69.088 111.506 90)
+		(property "Reference" "C8"
+			(at 69.596 121.158 90)
 			(effects
 				(font
@@
 		)
 		(property "Value" "1 nF"
-			(at 68.834 108.966 90)
-			(effects
-				(font
-					(size 1.27 1.27)
-				)
-				(justify left)
-			)
-		)
-		(property "Footprint" "Capacitor_SMD:C_01005_0402Metric"
+			(at 69.342 118.618 90)
+			(effects
+				(font
+					(size 1.27 1.27)
+				)
+				(justify left)
+			)
+		)
+		(property "Footprint" "Capacitor_SMD:C_0805_2012Metric"
 			(at 67.31 116.5352 0)
 			(effects
@@
 			(project "RFID_Reader"
 				(path "/4670be35-0898-46f4-be4d-f086d3203cc5/68791068-2e08-46a9-8a2f-80be28f652d5"
-					(reference "C20")
+					(reference "C8")
 					(unit 1)
 				)
@@
 		(on_board yes)
 		(dnp no)
-		(property "Reference" "C17"
+		(property "Reference" "CANT2"
 			(at 122.682 111.252 0)
 			(effects
@@
 			)
 		)
-		(property "Value" "Cant"
+		(property "Value" "tbd"
 			(at 124.714 111.252 0)
 			(effects
@@
 			)
 		)
-		(property "Footprint" "Capacitor_SMD:C_01005_0402Metric"
+		(property "Footprint" "Capacitor_SMD:C_0805_2012Metric"
 			(at 123.19 111.4552 0)
 			(effects
@@
 			(project "RFID_Reader"
 				(path "/4670be35-0898-46f4-be4d-f086d3203cc5/68791068-2e08-46a9-8a2f-80be28f652d5"
-					(reference "C17")
+					(reference "CANT2")
 					(unit 1)
 				)
@@
 		(dnp no)
 		(fields_autoplaced yes)
-		(property "Reference" "L2"
+		(property "Reference" "L0B1"
 			(at 91.44 90.17 90)
 			(effects
@@
 			)
 		)
-		(property "Footprint" "Inductor_SMD:L_2010_5025Metric"
+		(property "Footprint" "Inductor_SMD:L_0805_2012Metric"
 			(at 91.44 95.25 0)
 			(effects
@@
 			(project "RFID_Reader"
 				(path "/4670be35-0898-46f4-be4d-f086d3203cc5/68791068-2e08-46a9-8a2f-80be28f652d5"
-					(reference "L2")
+					(reference "L0B1")
 					(unit 1)
 				)
@@
 		(on_board yes)
 		(dnp no)
-		(property "Reference" "R9"
+		(property "Reference" "R1B1"
 			(at 97.536 101.092 90)
 			(effects
@@
 			)
 		)
-		(property "Footprint" "Resistor_SMD:R_01005_0402Metric"
+		(property "Footprint" "Resistor_SMD:R_0805_2012Metric"
 			(at 105.918 100.33 90)
 			(effects
@@
 			(project "RFID_Reader"
 				(path "/4670be35-0898-46f4-be4d-f086d3203cc5/68791068-2e08-46a9-8a2f-80be28f652d5"
-					(reference "R9")
+					(reference "R1B1")
 					(unit 1)
 				)
@@
 		(on_board yes)
 		(dnp no)
-		(property "Reference" "C11"
+		(property "Reference" "C0B1"
 			(at 105.41 88.138 0)
 			(effects
@@
 			)
 		)
-		(property "Footprint" "Capacitor_SMD:C_01005_0402Metric"
+		(property "Footprint" "Capacitor_SMD:C_0805_2012Metric"
 			(at 96.8248 85.09 0)
 			(effects
@@
 			(project "RFID_Reader"
 				(path "/4670be35-0898-46f4-be4d-f086d3203cc5/68791068-2e08-46a9-8a2f-80be28f652d5"
-					(reference "C11")
-					(unit 1)
-				)
+					(reference "C0B1")
+					(unit 1)
+				)
